File: Cansat.sch (KiCad schematic (older format))
At the start: 3 parts

Commit message: E.E. additions
Additions I've made since two weeks ago??
Parts:
- removed VR1234?: VoltageRegulator, symbol Cansatfunsymbols:VoltageRegulator
- added 5VReg?: MAX8881_5V_REG, symbol MAX8881_5V_REG
- added Bar-Pres-Sensor?: MS5607, symbol MS5607
- added GPS?: Ublox, symbol Ublox
- added IC?: BNO055, BNO055, symbol BNO055
- added MAS803Q?: SPKR105dB, symbol SPKR105dB
- added Radio?: XBEE-PRO, symbol XBEE-PRO
- added SNAP2?: ERPM, symbol ERPM
- added SNAP?: SERVO, symbol SERVO
- added TDK-Lambda_CC1R5-0503SR-E?: 3.3vREG, symbol 3.3vREG
- added Temp-R?: NTC-LE203, symbol NTC-LE203
Connections:
- net labels removed: GNDA
Changed lines of the file:
@@
-EESchema Schematic File Version 4
-EELAYER 26 0
+EESchema Schematic File Version 2
+LIBS:power
+LIBS:device
+LIBS:transistors
+LIBS:conn
+LIBS:linear
+LIBS:regul
+LIBS:74xx
+LIBS:cmos4000
+LIBS:adc-dac
+LIBS:memory
+LIBS:xilinx
+LIBS:microcontrollers
+LIBS:dsp
+LIBS:microchip
+LIBS:analog_switches
+LIBS:motorola
+LIBS:texas
+LIBS:intel
+LIBS:audio
+LIBS:interface
+LIBS:digital-audio
+LIBS:philips
+LIBS:display
+LIBS:cypress
+LIBS:siliconi
+LIBS:opto
+LIBS:atmel
+LIBS:contrib
+LIBS:valves
+LIBS:Cansat-cache
+EELAYER 25 0
 EELAYER END
 $Descr A4 11693 8268
@@
 $EndComp
 $Comp
-L Cansatfunsymbols:VoltageRegulator VR1234?
-U 1 1 5BFE1269
-P 7600 1850
-F 0 "VR1234?" H 7625 1287 50  0000 C CNN
-F 1 "VoltageRegulator" H 7625 1196 50  0000 C CNN
-F 2 "" H 7550 1900 50  0001 C CNN
-F 3 "" H 7550 1900 50  0001 C CNN
-	1    7600 1850
+L BNO055 IC?
+U 1 1 5C58FCE6
+P 8150 3700
+F 0 "IC?" H 9700 4400 50  0000 L CNN
+F 1 "BNO055" H 9700 4300 50  0000 L CNN
+F 2 "BNO055" H 9700 4200 50  0001 L CNN
+F 3 "https://componentsearchengine.com/Datasheets/1/BNO055.pdf" H 9700 4100 50  0001 L CNN
+F 4 "IMUs - Inertial Measurement Units Absolute Orientation 9-Axis Sensor" H 9700 4000 50  0001 L CNN "Description"
+F 5 "1" H 9700 3900 50  0001 L CNN "Height"
+F 6 "262-BNO055" H 9700 3800 50  0001 L CNN "Mouser Part Number"
+F 7 "Bosch Sensortec" H 9700 3700 50  0001 L CNN "Manufacturer_Name"
+F 8 "BNO055" H 9700 3600 50  0001 L CNN "Manufacturer_Part_Number"
+	1    8150 3700
 	1    0    0    -1
 $EndComp
 $Comp
-L power:GNDA #PWR?
-U 1 1 5BFE141D
-P 7600 2150
-F 0 "#PWR?" H 7600 1900 50  0001 C CNN
-F 1 "GNDA" H 7605 1977 50  0000 C CNN
-F 2 "" H 7600 2150 50  0001 C CNN
-F 3 "" H 7600 2150 50  0001 C CNN
-	1    7600 2150
+L ERPM SNAP2?
+U 1 1 5C58FDF0
+P 1950 4750
+F 0 "SNAP2?" H 1970 4310 60  0000 C CNN
+F 1 "ERPM" H 1830 5230 60  0000 L CNN
+F 2 "" H 1950 4750 60  0001 C CNN
+F 3 "" H 1950 4750 60  0001 C CNN
+	1    1950 4750
 	1    0    0    -1
 $EndComp
+$Comp
+L MS5607 Bar-Pres-Sensor?
+U 1 1 5C59014C
+P 2000 2250
+F 0 "Bar-Pres-Sensor?" H 1580 2570 60  0000 L BNN
+F 1 "MS5607" H 2000 1790 60  0000 C CNN
+F 2 "" H 2000 2250 60  0001 C CNN
+F 3 "" H 2000 2250 60  0001 C CNN
+	1    2000 2250
+	0    -1   -1   0
+$EndComp
+$Comp
+L NTC-LE203 Temp-R?
+U 1 1 5C5901BF
+P 1900 3850
+F 0 "Temp-R?" H 1890 3720 60  0000 C CNN
+F 1 "NTC-LE203" H 1670 3980 60  0000 L BNN
+F 2 "" H 1670 3980 60  0001 C CNN
+F 3 "" H 1670 3980 60  0001 C CNN
+	1    1900 3850
+	1    0    0    -1
+$EndComp
+$Comp
+L SERVO SNAP?
+U 1 1 5C590266
+P 1850 6300
+F 0 "SNAP?" H 1960 6570 60  0000 C CNN
+F 1 "SERVO" H 1720 6790 60  0000 L CNN
+F 2 "" H 1850 6300 60  0001 C CNN
+F 3 "" H 1850 6300 60  0001 C CNN
+	1    1850 6300
+	1    0    0    -1
+$EndComp
+$Comp
+L XBEE-PRO Radio?
+U 1 1 5C5903B1
+P 7100 5150
+F 0 "Radio?" H 7930 4220 60  0000 C CNN
+F 1 "XBEE-PRO" H 7310 6310 60  0000 L BNN
+F 2 "" H 7100 5150 60  0001 C CNN
+F 3 "" H 7100 5150 60  0001 C CNN
+	1    7100 5150
+	1    0    0    -1
+$EndComp
+$Comp
+L SPKR105dB MAS803Q?
+U 1 1 5C591308
+P 10200 1500
+F 0 "MAS803Q?" H 9830 1460 98  0000 L BNN
+F 1 "SPKR105dB" H 10222 960 60  0000 C CNN
+F 2 "" H 10200 1500 60  0001 C CNN
+F 3 "" H 10200 1500 60  0001 C CNN
+	1    10200 1500
+	1    0    0    -1
+$EndComp
+$Comp
+L Ublox GPS?
+U 1 1 5C5E6F41
+P 9050 5550
+F 0 "GPS?" H 9055 5540 60  0000 C CNN
+F 1 "Ublox" H 9035 5880 60  0000 C CNN
+F 2 "" H 9055 5540 60  0001 C CNN
+F 3 "" H 9055 5540 60  0001 C CNN
+	1    9050 5550
+	1    0    0    -1
+$EndComp
+$Comp
+L MAX8881_5V_REG 5VReg?
+U 1 1 5C60EFCC
+P 8300 1250
+F 0 "5VReg?" H 8295 1610 60  0000 C CNN
+F 1 "MAX8881_5V_REG" H 8315 985 60  0000 C CNN
+F 2 "" H 8295 1610 60  0001 C CNN
+F 3 "" H 8295 1610 60  0001 C CNN
+	1    8300 1250
+	1    0    0    -1
+$EndComp
+$Comp
+L 3.3vREG TDK-Lambda_CC1R5-0503SR-E?
+U 1 1 5C60F046
+P 7000 1350
+F 0 "TDK-Lambda_CC1R5-0503SR-E?" H 7020 700 60  0000 C CNN
+F 1 "3.3vREG" H 7015 1970 60  0000 C CNN
+F 2 "" H 6975 1310 60  0001 C CNN
+F 3 "" H 6975 1310 60  0001 C CNN
+	1    7000 1350
+	1    0    0    -1
+$EndComp

Commit message: attempt schematic
this needs work
Connections:
- net labels added: 3V_IN, 3V_OUT, 5V_OUT, 6V_IN, 6V_Out, GND
- wire segments 0 -> 109
Other:
- moved on the sheet: 5VReg?, Bar-Pres-Sensor?

Commit message: Found a more accurate Xmega schema from mouser.com
updated schematic
Parts:
- removed U?: ATxmega128A1U-AU, Package_QFP:TQFP-100_14x14mm_P0.5mm, symbol MCU_Microchip_ATmega:ATxmega128A1U-AU
- added IC?: ATXMEGA128A4U-AU, QFP80P1200X1200X120-44N, symbol ATXMEGA128A4U-AU
Connections:
- net labels added: 3.3V_IN, 3.3V_OUT, ADC_Pin, MCU_MOSFET?Pin
- net labels removed: 3V_IN, 3V_OUT
- wire segments 109 -> 75
Other:
- moved on the sheet: Bar-Pres-Sensor?, GPS?, SNAP?, Temp-R?

Commit message: "offical" schematic and footprints found
more updates
Parts:
- removed Radio?: XBEE-PRO, symbol XBEE-PRO
- removed SNAP2?: ERPM, symbol ERPM
- added IC?: XBP9B-XCWT-001, XBP9BXCWT001, symbol XBP9B-XCWT-001
- added IC?: SFH_7776, SFH7776, symbol SFH_7776
Connections:
- wire segments 75 -> 95
Other:
- moved on the sheet: GPS?
Changed lines of the file:
@@
-$EndComp
-$Comp
-L ERPM SNAP2?
-U 1 1 5C58FDF0
-P 5340 1215
-F 0 "SNAP2?" H 5360 775 60  0000 C CNN
-F 1 "ERPM" H 5220 1695 60  0000 L CNN
-F 2 "" H 5340 1215 60  0001 C CNN
-F 3 "" H 5340 1215 60  0001 C CNN
-	1    5340 1215
-	1    0    0    -1
 $EndComp
 $Comp
@@
 $EndComp
 $Comp
-L XBEE-PRO Radio?
-U 1 1 5C5903B1
-P 6410 5065
-F 0 "Radio?" H 7240 4135 60  0000 C CNN
-F 1 "XBEE-PRO" H 6620 6225 60  0000 L BNN
-F 2 "" H 6410 5065 60  0001 C CNN
-F 3 "" H 6410 5065 60  0001 C CNN
-	1    6410 5065
-	1    0    0    -1
-$EndComp
-$Comp
 L SPKR105dB MAS803Q?
 U 1 1 5C591308
@@
 	1    0    0    -1
 $EndComp
-Text GLabel 5040 1165 0    60   Input ~ 0
+Text GLabel 5860 2420 0    60   Input ~ 0
 3.3V_IN
 Text GLabel 3135 925  0    60   Input ~ 0
@@
 Text GLabel 4315 3485 2    60   Input ~ 0
 3.3V_IN
-Text GLabel 2560 6670 2    60   Input ~ 0
-3.3V_IN
-Text GLabel 7155 4655 2    60   Input ~ 0
+Text GLabel 2020 2100 2    60   Input ~ 0
+3.3V_IN
+Text GLabel 1575 5305 2    60   Input ~ 0
 3.3V_IN
 Text GLabel 7950 3800 0    60   Input ~ 0
@@
 Text GLabel 8295 3190 3    60   UnSpc ~ 0
 GND
-Text GLabel 5615 4665 0    60   UnSpc ~ 0
-GND
-Text GLabel 2565 6315 2    60   UnSpc ~ 0
+Text GLabel 1840 6620 2    60   UnSpc ~ 0
+GND
+Text GLabel 2025 1745 2    60   UnSpc ~ 0
 GND
 Text GLabel 10920 5400 2    60   UnSpc ~ 0
 GND
-Text GLabel 5095 1465 0    60   UnSpc ~ 0
+Text GLabel 5800 2620 0    60   UnSpc ~ 0
 GND
 Text GLabel 4355 3745 0    60   UnSpc ~ 0
@@
 L Ublox GPS?
 U 1 1 5C5E6F41
-P 1630 6550
-F 0 "GPS?" H 1635 6540 60  0000 C CNN
-F 1 "Ublox" H 1615 6880 60  0000 C CNN
-F 2 "" H 1635 6540 60  0001 C CNN
-F 3 "" H 1635 6540 60  0001 C CNN
-	1    1630 6550
+P 1090 1980
+F 0 "GPS?" H 1095 1970 60  0000 C CNN
+F 1 "Ublox" H 1075 2310 60  0000 C CNN
+F 2 "" H 1095 1970 60  0001 C CNN
+F 3 "" H 1095 1970 60  0001 C CNN
+	1    1090 1980
 	1    0    0    -1
 $EndComp
@@
 	3720 1035 4125 1035
 Wire Wire Line
-	5315 1155 5040 1165
-Wire Wire Line
 	10880 5675 10920 5400
 Wire Wire Line
 	10700 5675 10455 5400
-Connection ~ 2565 6315
-Connection ~ 2560 6670
+Connection ~ 2025 1745
+Connection ~ 2020 2100
 Wire Wire Line
 	1520 965  1775 965
@@
 	1775 965  1775 895
 Wire Wire Line
-	5315 1240 5340 1240
-Wire Wire Line
-	5340 1240 5340 1465
-Wire Wire Line
-	5340 1465 5095 1465
-Wire Wire Line
-	1450 6620 1535 6620
-Wire Wire Line
-	1490 6130 1490 6620
-Wire Wire Line
-	1490 6130 2155 6130
-Wire Wire Line
-	2155 6130 2155 6315
-Wire Wire Line
-	2155 6315 2565 6315
-Wire Wire Line
-	1450 6585 1490 6585
-Connection ~ 1490 6585
-Wire Wire Line
-	1450 6510 1490 6510
-Connection ~ 1490 6510
-Wire Wire Line
-	1450 6470 1490 6470
-Connection ~ 1490 6470
-Wire Wire Line
-	1450 6350 1490 6350
-Connection ~ 1490 6350
-Wire Wire Line
-	1450 6310 1490 6310
-Connection ~ 1490 6310
-Wire Wire Line
-	1785 6430 1810 6430
-Wire Wire Line
-	1785 6130 1785 6670
-Connection ~ 1785 6130
-Wire Wire Line
-	1810 6390 1785 6390
-Connection ~ 1785 6390
-Wire Wire Line
-	1810 6350 1785 6350
-Connection ~ 1785 6350
-Wire Wire Line
-	1810 6310 1785 6310
-Connection ~ 1785 6310
-Wire Wire Line
-	1785 6670 1810 6670
-Connection ~ 1785 6430
-Wire Wire Line
-	1810 6630 1785 6630
-Connection ~ 1785 6630
-Wire Wire Line
-	1810 6470 1745 6470
-Wire Wire Line
-	1745 6470 1745 6850
-Wire Wire Line
-	1745 6850 2560 6850
-Wire Wire Line
-	2560 6850 2560 6670
-Wire Wire Line
-	1810 6790 1745 6790
-Connection ~ 1745 6790
-Wire Wire Line
-	1535 6620 1535 6810
-Connection ~ 1490 6620
-Wire Wire Line
-	1715 6810 1715 6760
-Wire Wire Line
-	1715 6760 1535 6760
-Connection ~ 1535 6760
-Wire Wire Line
-	6720 4655 7160 4655
-Wire Wire Line
-	6020 4655 5615 4655
-Wire Wire Line
-	5615 4655 5615 4665
-Wire Wire Line
-	3650 3485 4315 3485
+	910  2050 950  2050
+Wire Wire Line
+	950  2050 995  2050
+Wire Wire Line
+	950  1560 950  1740
+Wire Wire Line
+	950  1740 950  1780
+Wire Wire Line
+	950  1780 950  1900
+Wire Wire Line
+	950  1900 950  1940
+Wire Wire Line
+	950  1940 950  2015
+Wire Wire Line
+	950  2015 950  2050
+Wire Wire Line
+	950  1560 1245 1560
+Wire Wire Line
+	1245 1560 1615 1560
+Wire Wire Line
+	1615 1560 1615 1745
+Wire Wire Line
+	1615 1745 2025 1745
+Wire Wire Line
+	910  2015 950  2015
+Connection ~ 950  2015
+Wire Wire Line
+	910  1940 950  1940
+Connection ~ 950  1940
+Wire Wire Line
+	910  1900 950  1900
+Connection ~ 950  1900
+Wire Wire Line
+	910  1780 950  1780
+Connection ~ 950  1780
+Wire Wire Line
+	910  1740 950  1740
+Connection ~ 950  1740
+Wire Wire Line
+	1245 1860 1270 1860
+Wire Wire Line
+	1245 1560 1245 1740
+Wire Wire Line
+	1245 1740 1245 1780
+Wire Wire Line
+	1245 1780 1245 1820
+Wire Wire Line
+	1245 1820 1245 1860
+Wire Wire Line
+	1245 1860 1245 2060
+Wire Wire Line
+	1245 2060 1245 2100
+Connection ~ 1245 1560
+Wire Wire Line
+	1270 1820 1245 1820
+Connection ~ 1245 1820
+Wire Wire Line
+	1270 1780 1245 1780
+Connection ~ 1245 1780
+Wire Wire Line
+	1270 1740 1245 1740
+Connection ~ 1245 1740
+Wire Wire Line
+	1245 2100 1270 2100
+Connection ~ 1245 1860
+Wire Wire Line
+	1270 2060 1245 2060
+Connection ~ 1245 2060
+Wire Wire Line
+	1270 1900 1205 1900
+Wire Wire Line
+	1205 1900 1205 2220
+Wire Wire Line
+	1205 2220 1205 2280
+Wire Wire Line
+	1205 2280 2020 2280
+Wire Wire Line
+	2020 2280 2020 2100
+Wire Wire Line
+	1270 2220 1205 2220
+Connection ~ 1205 2220
+Wire Wire Line
+	995  2050 995  2190
+Wire Wire Line
+	995  2190 995  2240
+Connection ~ 950  2050
+Wire Wire Line
+	1175 2240 1175 2190
+Wire Wire Line
+	1175 2190 995  2190
+Connection ~ 995  2190
+Wire Wire Line
+	1580 5505 1575 5305
+Wire Wire Line
+	3650 3485 4025 3485
+Wire Wire Line
+	4025 3485 4315 3485
 Wire Wire Line
 	8950 3000 8950 2925
@@
 $EndComp
 Wire Wire Line
-	4355 5200 4355 3585
+	4355 5200 4355 3745
+Wire Wire Line
+	4355 3745 4355 3585
 Wire Wire Line
 	4355 3585 3650 3585
@@
 	2950 4985 2950 5200
 Wire Wire Line
-	1660 5200 4355 5200
+	1660 5200 2950 5200
+Wire Wire Line
+	2950 5200 4355 5200
 Wire Wire Line
 	2050 3985 1660 3985
@@
 Wire Wire Line
 	6240 1655 6240 1660
+$Comp
+L XBP9B-XCWT-001 IC?
+U 1 1 5C6605C9
+P 4440 5765
+F 0 "IC?" H 4410 6080 50  0000 L CNN
+F 1 "XBP9B-XCWT-001" H 4070 5575 50  0000 L CNN
+F 2 "XBP9BXCWT001" H 4180 4210 50  0001 L CNN
+F 3 "http://www.mouser.com/datasheet/2/111/ds_xbeeproxsc-794439.pdf" H 3380 4310 50  0001 L CNN
+F 4 "RF Modules Xbee-PRO XSC S3B 900MHz, 250mW Wire" H 3420 4390 50  0001 L CNN "Description"
+F 5 "2.79" H 7535 5855 50  0001 L CNN "Height"
+F 6 "888-XBP9B-XCWT-001" H 3995 4500 50  0001 L CNN "Mouser Part Number"
+F 7 "Digi International" H 4205 4135 50  0001 L CNN "Manufacturer_Name"
+F 8 "XBP9B-XCWT-001" H 4180 4045 50  0001 L CNN "Manufacturer_Part_Number"
+	1    4440 5765
+	1    0    0    -1
+$EndComp
+Wire Wire Line
+	1580 6405 1580 6620
+Wire Wire Line
+	1580 6620 1840 6620
+$Comp
+L SFH_7776 IC?
+U 1 1 5C66198F
+P 6730 2460
+F 0 "IC?" H 6745 2545 50  0000 L CNN
+F 1 "SFH_7776" H 6615 2345 50  0000 L CNN
+F 2 "SFH7776" H 6605 1870 50  0001 L CNN
+F 3 "https://www.arrow.com/en/products/sfh7776/osram-opto-semiconductors" H 5775 1710 50  0001 L CNN
+F 4 "SFH 7776 Osram Opto Ambient Light and Proximity Sensor Surface Mount 8-Pin Miniature" H 5765 1620 50  0001 L CNN "Description"
+F 5 "1.45" H 7245 2295 50  0001 L CNN "Height"
+F 6 "720-SFH7776" H 6515 1795 50  0001 L CNN "Mouser Part Number"
+F 7 "OSRAM Opto Semiconductors" H 6195 1530 50  0001 L CNN "Manufacturer_Name"
+F 8 "SFH 7776" H 6585 1445 50  0001 L CNN "Manufacturer_Part_Number"
+	1    6730 2460
+	1    0    0    -1
+$EndComp
+Wire Wire Line
+	6195 2425 5860 2425
+Wire Wire Line
+	5860 2425 5860 2420
+Wire Wire Line
+	6195 2625 5800 2625
+Wire Wire Line
+	5800 2625 5800 2620
+Wire Wire Line
+	7395 2425 7395 2525
+Wire Wire Line
+	7395 2525 7395 2525
+Wire Wire Line
+	7395 2425 7395 2425
 $EndSCHEMATC

Commit message: Continued adding common components
Parts:
- added CAP? (x4): Capacitor, symbol Capacitor
- added RES? (x3): Resistor, symbol Resistor
Connections:
- net labels added: I2C_clk, I2C_serialdata, Vint, Vint,up, Vio
- wire segments 95 -> 125
Other:
- moved on the sheet: IC?
Changed lines of the file:
@@
 L BNO055 IC?
 U 1 1 5C58FCE6
-P 8150 3700
-F 0 "IC?" H 9700 4400 50  0000 L CNN
-F 1 "BNO055" H 9700 4300 50  0000 L CNN
-F 2 "BNO055" H 9700 4200 50  0001 L CNN
-F 3 "https://componentsearchengine.com/Datasheets/1/BNO055.pdf" H 9700 4100 50  0001 L CNN
-F 4 "IMUs - Inertial Measurement Units Absolute Orientation 9-Axis Sensor" H 9700 4000 50  0001 L CNN "Description"
-F 5 "1" H 9700 3900 50  0001 L CNN "Height"
-F 6 "262-BNO055" H 9700 3800 50  0001 L CNN "Mouser Part Number"
-F 7 "Bosch Sensortec" H 9700 3700 50  0001 L CNN "Manufacturer_Name"
-F 8 "BNO055" H 9700 3600 50  0001 L CNN "Manufacturer_Part_Number"
-	1    8150 3700
+P 6790 3640
+F 0 "IC?" H 8340 4340 50  0000 L CNN
+F 1 "BNO055" H 8340 4240 50  0000 L CNN
+F 2 "BNO055" H 8340 4140 50  0001 L CNN
+F 3 "https://componentsearchengine.com/Datasheets/1/BNO055.pdf" H 8340 4040 50  0001 L CNN
+F 4 "IMUs - Inertial Measurement Units Absolute Orientation 9-Axis Sensor" H 8340 3940 50  0001 L CNN "Description"
+F 5 "1" H 8340 3840 50  0001 L CNN "Height"
+F 6 "262-BNO055" H 8340 3740 50  0001 L CNN "Mouser Part Number"
+F 7 "Bosch Sensortec" H 8340 3640 50  0001 L CNN "Manufacturer_Name"
+F 8 "BNO055" H 8340 3540 50  0001 L CNN "Manufacturer_Part_Number"
+	1    6790 3640
 	1    0    0    -1
 $EndComp
@@
 	1    0    0    -1
 $EndComp
-Text GLabel 5860 2420 0    60   Input ~ 0
+Text GLabel 3020 6765 0    60   Output ~ 0
 3.3V_IN
 Text GLabel 3135 925  0    60   Input ~ 0
@@
 Text GLabel 1575 5305 2    60   Input ~ 0
 3.3V_IN
-Text GLabel 7950 3800 0    60   Input ~ 0
+Text GLabel 6590 3740 0    60   Input ~ 0
 3.3V_IN
 Text GLabel 10200 1760 0    60   Input ~ 0
@@
 Text GLabel 9610 6100 0    60   UnSpc ~ 0
 GND
-Text GLabel 8295 3190 3    60   UnSpc ~ 0
+Text GLabel 6935 3130 3    60   UnSpc ~ 0
 GND
 Text GLabel 1840 6620 2    60   UnSpc ~ 0
@@
 Text GLabel 10920 5400 2    60   UnSpc ~ 0
 GND
-Text GLabel 5800 2620 0    60   UnSpc ~ 0
+Text GLabel 2825 7020 0    60   UnSpc ~ 0
 GND
 Text GLabel 4355 3745 0    60   UnSpc ~ 0
@@
 	4025 3485 4315 3485
 Wire Wire Line
-	8950 3000 8950 2925
-Wire Wire Line
-	8950 2925 8295 2925
-Wire Wire Line
-	8295 2925 8295 3190
-Wire Wire Line
-	8150 3700 8150 3190
-Wire Wire Line
-	8150 3190 8295 3190
-Wire Wire Line
-	8150 3800 7950 3800
+	7590 2940 7590 2865
+Wire Wire Line
+	7590 2865 6935 2865
+Wire Wire Line
+	6935 2865 6935 3130
+Wire Wire Line
+	6790 3640 6790 3130
+Wire Wire Line
+	6790 3130 6935 3130
+Wire Wire Line
+	6790 3740 6590 3740
 $Comp
 L ATXMEGA128A4U-AU IC?
@@
 L SFH_7776 IC?
 U 1 1 5C66198F
-P 6730 2460
-F 0 "IC?" H 6745 2545 50  0000 L CNN
-F 1 "SFH_7776" H 6615 2345 50  0000 L CNN
-F 2 "SFH7776" H 6605 1870 50  0001 L CNN
-F 3 "https://www.arrow.com/en/products/sfh7776/osram-opto-semiconductors" H 5775 1710 50  0001 L CNN
-F 4 "SFH 7776 Osram Opto Ambient Light and Proximity Sensor Surface Mount 8-Pin Miniature" H 5765 1620 50  0001 L CNN "Description"
-F 5 "1.45" H 7245 2295 50  0001 L CNN "Height"
-F 6 "720-SFH7776" H 6515 1795 50  0001 L CNN "Mouser Part Number"
-F 7 "OSRAM Opto Semiconductors" H 6195 1530 50  0001 L CNN "Manufacturer_Name"
-F 8 "SFH 7776" H 6585 1445 50  0001 L CNN "Manufacturer_Part_Number"
-	1    6730 2460
-	1    0    0    -1
-$EndComp
-Wire Wire Line
-	6195 2425 5860 2425
-Wire Wire Line
-	5860 2425 5860 2420
-Wire Wire Line
-	6195 2625 5800 2625
-Wire Wire Line
-	5800 2625 5800 2620
-Wire Wire Line
-	7395 2425 7395 2525
-Wire Wire Line
-	7395 2525 7395 2525
-Wire Wire Line
-	7395 2425 7395 2425
+P 4215 6845
+F 0 "IC?" H 4230 6930 50  0000 L CNN
+F 1 "SFH_7776" H 4100 6730 50  0000 L CNN
+F 2 "SFH7776" H 4090 6255 50  0001 L CNN
+F 3 "https://www.arrow.com/en/products/sfh7776/osram-opto-semiconductors" H 3260 6095 50  0001 L CNN
+F 4 "SFH 7776 Osram Opto Ambient Light and Proximity Sensor Surface Mount 8-Pin Miniature" H 3250 6005 50  0001 L CNN "Description"
+F 5 "1.45" H 4730 6680 50  0001 L CNN "Height"
+F 6 "720-SFH7776" H 4000 6180 50  0001 L CNN "Mouser Part Number"
+F 7 "OSRAM Opto Semiconductors" H 3680 5915 50  0001 L CNN "Manufacturer_Name"
+F 8 "SFH 7776" H 4070 5830 50  0001 L CNN "Manufacturer_Part_Number"
+	1    4215 6845
+	1    0    0    -1
+$EndComp
+Wire Wire Line
+	3510 6775 3680 6775
+Wire Wire Line
+	3510 6775 3340 6770
+Wire Wire Line
+	3340 6770 3330 6770
+Wire Wire Line
+	3330 6770 3020 6765
+Wire Wire Line
+	3330 7020 3515 7020
+Wire Wire Line
+	3515 7020 3535 7020
+Wire Wire Line
+	3340 7010 3330 7020
+Wire Wire Line
+	3115 7010 3280 7010
+Wire Wire Line
+	3280 7010 3340 7010
+Wire Wire Line
+	3115 7010 2825 7020
+Wire Wire Line
+	4880 6810 4880 6910
+$Comp
+L Capacitor CAP?
+U 1 1 5C66264C
+P 3330 6895
+F 0 "CAP?" H 3345 7165 12  0000 C CNN
+F 1 "Capacitor" H 3425 6910 60  0000 C CNN
+F 2 "" H 3330 6895 60  0001 C CNN
+F 3 "" H 3330 6895 60  0001 C CNN
+	1    3330 6895
+	1    0    0    -1
+$EndComp
+$Comp
+L Capacitor CAP?
+U 1 1 5C6639D6
+P 3515 6895
+F 0 "CAP?" H 3530 7165 60  0000 C CNN
+F 1 "Capacitor" H 3425 6910 60  0000 C CNN
+F 2 "" H 3515 6895 60  0001 C CNN
+F 3 "" H 3515 6895 60  0001 C CNN
+	1    3515 6895
+	1    0    0    -1
+$EndComp
+$Comp
+L Resistor RES?
+U 1 1 5C663E1F
+P 3585 7480
+F 0 "RES?" V 3595 7670 60  0000 C CNN
+F 1 "Resistor" V 3725 7675 60  0000 C CNN
+F 2 "" H 3585 7480 60  0001 C CNN
+F 3 "" H 3585 7480 60  0001 C CNN
+	1    3585 7480
+	0    1    1    0
+$EndComp
+$Comp
+L Resistor RES?
+U 1 1 5C663F58
+P 4885 7465
+F 0 "RES?" V 4845 7645 60  0000 C CNN
+F 1 "Resistor" V 4720 7665 60  0000 C CNN
+F 2 "" H 4885 7465 60  0001 C CNN
+F 3 "" H 4885 7465 60  0001 C CNN
+	1    4885 7465
+	0    -1   -1   0
+$EndComp
+Text GLabel 3530 7620 0    60   Output ~ 0
+Vio
+Wire Wire Line
+	3585 7560 4885 7560
+Wire Wire Line
+	4885 7560 4885 7545
+Wire Wire Line
+	4885 7385 4885 7110
+Wire Wire Line
+	4885 7110 4880 7110
+Wire Wire Line
+	3575 7295 3585 7400
+Wire Wire Line
+	3580 7175 3645 7175
+Wire Wire Line
+	3645 7175 3645 6910
+Wire Wire Line
+	3645 6910 3680 6910
+Wire Wire Line
+	3530 7620 3585 7620
+Wire Wire Line
+	3585 7620 3585 7560
+Text GLabel 5140 6910 1    60   Output ~ 0
+Vint,up
+Wire Wire Line
+	3680 7110 3520 7110
+Wire Wire Line
+	3520 7110 3520 7245
+Wire Wire Line
+	3520 7245 3120 7245
+Wire Wire Line
+	3120 7245 2985 7245
+Wire Wire Line
+	2985 7245 2985 7225
+Wire Wire Line
+	2985 7225 3020 6765
+$Comp
+L Capacitor CAP?
+U 1 1 5C6673BC
+P 3120 7135
+F 0 "CAP?" H 3135 7405 60  0000 C CNN
+F 1 "Capacitor" H 3205 7135 60  0000 C CNN
+F 2 "" H 3120 7135 60  0001 C CNN
+F 3 "" H 3120 7135 60  0001 C CNN
+	1    3120 7135
+	1    0    0    1
+$EndComp
+$Comp
+L Capacitor CAP?
+U 1 1 5C667441
+P 3280 7135
+F 0 "CAP?" H 3135 7405 60  0000 C CNN
+F 1 "Capacitor" H 3205 7135 60  0000 C CNN
+F 2 "" H 3280 7135 60  0001 C CNN
+F 3 "" H 3280 7135 60  0001 C CNN
+	1    3280 7135
+	1    0    0    1
+$EndComp
+Text GLabel 5035 7105 3    60   Output ~ 0
+Vint
+$Comp
+L Resistor RES?
+U 1 1 5C667FB7
+P 5140 6990
+F 0 "RES?" V 5165 6750 60  0000 C CNN
+F 1 "Resistor" V 5065 6745 60  0000 C CNN
+F 2 "" H 5140 6990 60  0001 C CNN
+F 3 "" H 5140 6990 60  0001 C CNN
+	1    5140 6990
+	0    -1   -1   0
+$EndComp
+Wire Wire Line
+	4880 7010 5035 7010
+Wire Wire Line
+	5035 7010 5035 7070
+Wire Wire Line
+	5035 7070 5035 7105
+Wire Wire Line
+	5140 7070 5035 7070
+Connection ~ 5035 7070
+Wire Wire Line
+	3680 6775 3680 6810
+Connection ~ 3330 7020
+Connection ~ 3280 7010
+Wire Wire Line
+	3535 7020 3680 7010
+Connection ~ 3515 7020
+Wire Wire Line
+	3330 6770 3330 6775
+Connection ~ 3330 6770
+Connection ~ 3510 6775
+Connection ~ 3115 7010
+Wire Wire Line
+	3120 7255 3120 7245
+Connection ~ 3120 7245
+Wire Wire Line
+	3120 7245 3280 7255
+Text GLabel 4885 7270 0    60   BiDi ~ 0
+I2C_serialdata
+Text GLabel 3575 7295 2    60   Input ~ 0
+I2C_clk
+Wire Wire Line
+	3580 7175 3575 7295
 $EndSCHEMATC

Commit message: Added in OpenLog Breakout
Parts:
- added Breakout?: OpenLog, symbol OpenLog
- added ML681_3V: Panasonic, symbol Device:Battery
- gave numbers to parts that had none: 2
Connections:
- net labels added: +3.3V, +3V, +5V, +6V, I2C_CLK
- net labels removed: 3.3V_IN, 6V_IN, 6V_Out
- wire segments 125 -> 84
Other:
- moved on the sheet: 5VReg?, CAP?, CoSel_SUS1R5, GPS?, IC?, OSRAM_IR, RES?, Temp-R?

Commit message: resized my mistake, again
Connections:
- net labels removed: I2C_CLK
- wire segments 84 -> 48
Other:
- moved on the sheet: Bar-Pres-Sensor?, GPS?, IC?

Commit message: new stuff 2.17.19
Parts:
- added SNAP?: FAN_0, symbol FAN_0
- added SNAP?: FAN_1, symbol FAN_1
- added comp?: VoltageDivider, symbol VoltageDivider
Connections:
- net labels added: ADC_Pin0, ADC_Pin1, MOSFET_0, MOSFET_1, MOSFET_2, SPI_CLK, SPI_INPUT, SPI_OUTPUT
- net labels removed: ADC_Pin
- wire segments 48 -> 72
Other:
- moved on the sheet: SNAP?
