File: Cansat.sch (KiCad schematic (older format))
At the start: 24 parts

Commit message: Finally: Footprint Library Created. CanSat_Dai_Atlas
lets see if it works
Parts:
- 5VReg?: symbol MAX8881_5V_REG -> Cansat-rescue:MAX8881_5V_REG
- Bar-Pres-Sensor?: symbol MS5607 -> Cansat-rescue:MS5607
- Breakout?: symbol OpenLog -> Cansat-rescue:OpenLog
- CAP? (x4): symbol Capacitor -> Cansat-rescue:Capacitor
- CoSel_SUS1R5: symbol 3.3vREG -> Cansat-rescue:3.3vREG
- GPS?: symbol Ublox -> Cansat-rescue:Ublox
- IC?: symbol BNO055 -> Cansat-rescue:BNO055
- IC?: symbol ATXMEGA128A4U-AU -> Cansat-rescue:ATXMEGA128A4U-AU
- IC?: symbol XBP9B-XCWT-001 -> Cansat-rescue:XBP9B-XCWT-001
- MAS803Q?: symbol SPKR105dB -> Cansat-rescue:SPKR105dB
- ML681_3V, surefire123A: symbol Device:Battery -> Cansat-rescue:Device_Battery
- OSRAM_IR: symbol SFH_7776 -> Cansat-rescue:SFH_7776
- RES? (x3): symbol Resistor -> Cansat-rescue:Resistor
- SNAP?: symbol SERVO -> Cansat-rescue:SERVO
- SNAP?: symbol FAN_0 -> Cansat-rescue:FAN_0
- SNAP?: symbol FAN_1 -> Cansat-rescue:FAN_1
- Temp-R?: symbol NTC-LE203 -> Cansat-rescue:NTC-LE203
- comp?: symbol VoltageDivider -> Cansat-rescue:VoltageDivider
Connections:
- wire segments 72 -> 78

Commit message: Placing Flags
Parts:
- added 100nF, 1uF, 4.7uF: C_Small, symbol Device:C_Small
- added D?: D_Small_ALT, symbol Device:D_Small_ALT
- added J?: XLR3_Switched, symbol Connector:XLR3_Switched
- gave numbers to parts that had none: 4
Connections:
- net labels added: 3V_OUT, 6V_OUT, ADC_PA0, ADC_PA1, Buzzer_ON_PD0, I2C_CLK_PC1, I2C_SD_PC0, LED_ON_PE0, USART_RX_PC2, USART_RX_PD2, USART_RX_PD6, USART_TX_PC3, USART_TX_PD3, USART_TX_PD7, VBUS
- net labels removed: ADC_Pin0, ADC_Pin1, I2C_clk, I2C_serialdata, MCU_MOSFET?Pin
- wire segments 78 -> 92
Changed lines of the file:
@@
 $EndComp
 Text GLabel 7752 646  0    60   Input ~ 0
-ADC_Pin0
+ADC_PA0
 Text GLabel 10200 1760 0    60   Input ~ 0
-MCU_MOSFET?Pin
-Text GLabel 7962 2237 0    60   Output ~ 0
+Buzzer_ON_PD0
+Text GLabel 7726 2434 0    60   Output ~ 0
 5V_OUT
 Text GLabel 8725 1069 2    60   Output ~ 0
@@
 $EndComp
 Wire Wire Line
-	7982 2087 7912 2087
-Wire Wire Line
-	7982 2152 7982 2237
-Wire Wire Line
-	7982 2237 7962 2237
+	7982 2087 7690 2087
+Wire Wire Line
+	7770 2283 7770 2284
+Wire Wire Line
+	7983 2153 7726 2434
 Wire Wire Line
 	8172 696  8167 651
@@
 	5881 821  5881 921
 $Comp
-L Cansat-rescue:Capacitor CAP?
+L Cansat-rescue:Capacitor 4.7uF
 U 1 1 5C66264C
 P 4331 906
-F 0 "CAP?" H 4346 1176 12  0000 C CNN
+F 0 "4.7uF" H 4346 1176 60  0000 C CNN
 F 1 "Capacitor" H 4426 921 60  0000 C CNN
 F 2 "" H 4331 906 60  0001 C CNN
@@
 $EndComp
 $Comp
-L Cansat-rescue:Capacitor CAP?
+L Cansat-rescue:Capacitor 100nF
 U 1 1 5C6639D6
 P 4516 906
-F 0 "CAP?" H 4531 1176 60  0000 C CNN
+F 0 "100nF" H 4617 1171 60  0000 C CNN
 F 1 "Capacitor" H 4426 921 60  0000 C CNN
 F 2 "" H 4516 906 60  0001 C CNN
@@
 $EndComp
 $Comp
-L Cansat-rescue:Resistor RES?
+L Cansat-rescue:Resistor 10K
 U 1 1 5C663E1F
 P 4586 1491
-F 0 "RES?" V 4596 1681 60  0000 C CNN
+F 0 "10K" V 4596 1681 60  0000 C CNN
 F 1 "Resistor" V 4726 1686 60  0000 C CNN
 F 2 "" H 4586 1491 60  0001 C CNN
@@
 $EndComp
 $Comp
-L Cansat-rescue:Resistor RES?
+L Cansat-rescue:Resistor 10K
 U 1 1 5C663F58
 P 5886 1476
-F 0 "RES?" V 5846 1656 60  0000 C CNN
+F 0 "10K" V 5846 1656 60  0000 C CNN
 F 1 "Resistor" V 5721 1676 60  0000 C CNN
 F 2 "" H 5886 1476 60  0001 C CNN
@@
 	3986 1256 3984 1254
 $Comp
-L Cansat-rescue:Capacitor CAP?
+L Cansat-rescue:Capacitor 4.7uF
 U 1 1 5C6673BC
 P 4121 1146
-F 0 "CAP?" H 4136 1416 60  0000 C CNN
+F 0 "4.7uF" H 4008 1420 60  0000 C CNN
 F 1 "Capacitor" H 4206 1146 60  0000 C CNN
 F 2 "" H 4121 1146 60  0001 C CNN
@@
 $EndComp
 $Comp
-L Cansat-rescue:Capacitor CAP?
+L Cansat-rescue:Capacitor 100nF
 U 1 1 5C667441
 P 4281 1146
-F 0 "CAP?" H 4136 1416 60  0000 C CNN
+F 0 "100nF" H 4296 1416 60  0000 C CNN
 F 1 "Capacitor" H 4206 1146 60  0000 C CNN
 F 2 "" H 4281 1146 60  0001 C CNN
@@
 Vint
 $Comp
-L Cansat-rescue:Resistor RES?
+L Cansat-rescue:Resistor 10k
 U 1 1 5C667FB7
 P 6141 1001
-F 0 "RES?" V 6166 761 60  0000 C CNN
+F 0 "10k" V 6166 761 60  0000 C CNN
 F 1 "Resistor" V 6066 756 60  0000 C CNN
 F 2 "" H 6141 1001 60  0001 C CNN
@@
 	4121 1265 3986 1256
 Text GLabel 5886 1281 0    60   BiDi ~ 0
-I2C_serialdata
+I2C_SD_PC0
 Text GLabel 4576 1306 2    60   Input ~ 0
-I2C_clk
+I2C_CLK_PC1
 Wire Wire Line
 	4581 1186 4576 1306
@@
 L power:GND #PWR?
 U 1 1 5C69A05C
-P 7912 2087
-F 0 "#PWR?" H 7912 1837 50  0001 C CNN
-F 1 "GND" H 7912 1937 50  0000 C CNN
-F 2 "" H 7912 2087 50  0000 C CNN
-F 3 "" H 7912 2087 50  0000 C CNN
-	1    7912 2087
+P 7690 2087
+F 0 "#PWR?" H 7690 1837 50  0001 C CNN
+F 1 "GND" H 7690 1937 50  0000 C CNN
+F 2 "" H 7690 2087 50  0000 C CNN
+F 3 "" H 7690 2087 50  0000 C CNN
+	1    7690 2087
 	0    1    1    0
 $EndComp
@@
 L power:+6V #PWR?
 U 1 1 5C69ABF6
-P 7982 2012
-F 0 "#PWR?" H 7982 1862 50  0001 C CNN
-F 1 "+6V" H 7982 2152 50  0000 C CNN
-F 2 "" H 7982 2012 50  0000 C CNN
-F 3 "" H 7982 2012 50  0000 C CNN
-	1    7982 2012
+P 7562 1994
+F 0 "#PWR?" H 7562 1844 50  0001 C CNN
+F 1 "+6V" H 7562 2134 50  0000 C CNN
+F 2 "" H 7562 1994 50  0000 C CNN
+F 3 "" H 7562 1994 50  0000 C CNN
+	1    7562 1994
 	0    -1   -1   0
 $EndComp
@@
 L power:GND #PWR?
 U 1 1 5C6A5131
-P 2103 1867
-F 0 "#PWR?" H 2103 1617 50  0001 C CNN
-F 1 "GND" H 2103 1717 50  0000 C CNN
-F 2 "" H 2103 1867 50  0000 C CNN
-F 3 "" H 2103 1867 50  0000 C CNN
-	1    2103 1867
+P 1765 1868
+F 0 "#PWR?" H 1765 1618 50  0001 C CNN
+F 1 "GND" H 1765 1718 50  0000 C CNN
+F 2 "" H 1765 1868 50  0000 C CNN
+F 3 "" H 1765 1868 50  0000 C CNN
+	1    1765 1868
 	0    1    1    0
 $EndComp
@@
 L power:+3.3V #PWR?
 U 1 1 5C6A5607
-P 2103 1418
-F 0 "#PWR?" H 2103 1268 50  0001 C CNN
-F 1 "+3.3V" H 2103 1558 50  0000 C CNN
-F 2 "" H 2103 1418 50  0000 C CNN
-F 3 "" H 2103 1418 50  0000 C CNN
-	1    2103 1418
+P 1779 1419
+F 0 "#PWR?" H 1779 1269 50  0001 C CNN
+F 1 "+3.3V" H 1779 1559 50  0000 C CNN
+F 2 "" H 1779 1419 50  0000 C CNN
+F 3 "" H 1779 1419 50  0000 C CNN
+	1    1779 1419
 	0    -1   -1   0
 $EndComp
@@
 $EndComp
 Text GLabel 8093 5735 2    60   Input ~ 0
-ADC_Pin1
+ADC_PA1
 $Comp
 L Cansat-rescue:FAN_0 SNAP?
@@
 Text GLabel 3016 1871 2    60   Input ~ 0
 SPI_OUTPUT
-Wire Wire Line
-	2120 1867 2120 1869
 $Comp
 L power:+3.3V #PWR?
@@
 	2102 1652 2102 1867
 Wire Wire Line
-	2102 1867 2120 1867
+	2102 1867 1766 1869
 Wire Wire Line
 	2204 2909 2370 2909
 Wire Wire Line
 	1851 2907 1851 2911
+$Comp
+L Device:C_Small 100nF
+U 1 1 5C6F9D3E
+P 1778 1640
+F 0 "100nF" H 1470 1694 50  0000 L CNN
+F 1 "C_Small" H 1376 1574 50  0000 L CNN
+F 2 "" H 1778 1640 50  0001 C CNN
+F 3 "~" H 1778 1640 50  0001 C CNN
+	1    1778 1640
+	1    0    0    -1
+$EndComp
+Wire Wire Line
+	1778 1740 1778 1869
+Wire Wire Line
+	1778 1869 1766 1869
+Wire Wire Line
+	1766 1869 1766 1868
+Connection ~ 1766 1869
+Wire Wire Line
+	1778 1540 1778 1419
+Wire Wire Line
+	1778 1419 1779 1419
+Wire Wire Line
+	2104 1419 2104 1420
+Connection ~ 1779 1419
+Wire Wire Line
+	1779 1419 2104 1419
+$Comp
+L Device:C_Small 1uF
+U 1 1 5C6FE128
+P 7770 1984
+F 0 "1uF" H 7940 1932 50  0000 R CNN
+F 1 "C_Small" H 7843 2054 50  0000 R CNN
+F 2 "" H 7770 1984 50  0001 C CNN
+F 3 "~" H 7770 1984 50  0001 C CNN
+	1    7770 1984
+	-1   0    0    1
+$EndComp
+$Comp
+L Device:C_Small 4.7uF
+U 1 1 5C6FE5E0
+P 7770 2184
+F 0 "4.7uF" H 7524 2124 50  0000 L CNN
+F 1 "C_Small" H 7700 2246 50  0000 L CNN
+F 2 "" H 7770 2184 50  0001 C CNN
+F 3 "~" H 7770 2184 50  0001 C CNN
+	1    7770 2184
+	1    0    0    -1
+$EndComp
+Wire Wire Line
+	7983 2012 7983 1885
+Wire Wire Line
+	7562 1885 7562 1994
+Wire Wire Line
+	7562 1885 7983 1885
+Connection ~ 7770 2284
+Wire Wire Line
+	7770 2284 7821 2331
+Wire Wire Line
+	8451 2157 7983 2157
+Wire Wire Line
+	7983 2157 7983 2153
+Wire Wire Line
+	7983 2151 7985 2151
+Connection ~ 7983 2153
+Wire Wire Line
+	7983 2153 7983 2151
+Connection ~ 7981 2011
+Text GLabel 9911 3776 3    50   Input ~ 0
+USART_RX_PC2
+Text GLabel 9996 3775 3    50   Output ~ 0
+USART_TX_PC3
+Text GLabel 3662 4441 0    60   Input ~ 0
+I2C_CLK_PC1
+Text GLabel 3662 4341 0    60   BiDi ~ 0
+I2C_SD_PC0
+Text GLabel 3962 5141 3    50   Input ~ 0
+USART_RX_PC2
+Text GLabel 4062 5141 3    50   Output ~ 0
+USART_TX_PC3
+Text GLabel 4962 5141 3    50   Input ~ 0
+USART_RX_PD2
+Text GLabel 5262 4441 2    50   Output ~ 0
+USART_TX_PD3
+Text GLabel 6414 6450 2    50   Input ~ 0
+USART_RX_PD2
+Text GLabel 6416 6296 2    50   Output ~ 0
+USART_TX_PD3
+Text GLabel 4762 5141 3    50   Output ~ 0
+Buzzer_ON_PD0
+Text GLabel 5262 3941 2    50   Output ~ 0
+LED_ON_PE0
+Text GLabel 4262 2541 1    60   Input ~ 0
+ADC_PA1
+Text GLabel 4362 2541 1    60   Input ~ 0
+ADC_PA0
+Text GLabel 1088 4347 0    50   Output ~ 0
+USART_TX_PD7
+Text GLabel 1083 4519 0    50   Input ~ 0
+USART_RX_PD6
+Text GLabel 5262 4141 2    50   Input ~ 0
+USART_RX_PD6
+Text GLabel 5262 4041 2    50   Output ~ 0
+USART_TX_PD7
+$Comp
+L power:VBUS #PWR?
+U 1 1 5C7191DB
+P 9172 5394
+F 0 "#PWR?" H 9172 5244 50  0001 C CNN
+F 1 "VBUS" V 9187 5521 50  0000 L CNN
+F 2 "" H 9172 5394 50  0001 C CNN
+F 3 "" H 9172 5394 50  0001 C CNN
+	1    9172 5394
+	0    -1   -1   0
+$EndComp
+$Comp
+L Connector:XLR3_Switched J?
+U 1 1 5C7196DF
+P 9472 5394
+F 0 "J?" H 9472 5759 50  0000 C CNN
+F 1 "XLR3_Switched" H 9472 5668 50  0000 C CNN
+F 2 "" H 9472 5494 50  0001 C CNN
+F 3 " ~" H 9472 5494 50  0001 C CNN
+	1    9472 5394
+	1    0    0    -1
+$EndComp
+Text GLabel 9772 5394 3    50   Output ~ 0
+6V_OUT
+Text GLabel 8853 5528 0    50   Output ~ 0
+3V_OUT
+$Comp
+L Device:D_Small_ALT D?
+U 1 1 5C71BBB3
+P 8853 5628
+F 0 "D?" V 8807 5696 50  0000 L CNN
+F 1 "D_Small_ALT" V 8898 5696 50  0000 L CNN
+F 2 "" V 8853 5628 50  0001 C CNN
+F 3 "~" V 8853 5628 50  0001 C CNN
+	1    8853 5628
+	0    1    1    0
+$EndComp
 $EndSCHEMATC

Commit message: more flags, R, CAPs
Parts:
- removed J?: XLR3_Switched, symbol Connector:XLR3_Switched
- added 100nF (x2), 120nF, 6.8nF: C_Small, symbol Device:C_Small
- added 10K? (x4): Resistor, symbol Cansat-rescue:Resistor
- added D?: D_Small_ALT, symbol Device:D_Small_ALT
- added Fan_0_CTRL, Fan_1_CTRL, Servo_CTRL: 2N7002, Package_TO_SOT_SMD:SOT-23, symbol Transistor_FET:2N7002
- added SW?: SW_SPDT_MSM, symbol Switch:SW_SPDT_MSM
- comp?: footprint (none) -> voltage_divider
Connections:
- wire segments 92 -> 128

Commit message: more tags, more components
Parts:
- gave numbers to parts that had none: 1
Connections:
- net labels added: nBootLoadPin, nResetPin
- wire segments 128 -> 152
Other:
- moved on the sheet: 10K?, 10K?opt
Changed lines of the file:
@@
 U 1 1 5C58FCE6
 P 6790 3640
-F 0 "IC?" H 8340 4340 50  0000 L CNN
-F 1 "BNO055" H 8340 4240 50  0000 L CNN
+F 0 "IC?" H 7830 3644 50  0000 L CNN
+F 1 "BNO055" H 7734 3716 50  0000 L CNN
 F 2 "BNO055" H 8340 4140 50  0001 L CNN
 F 3 "https://componentsearchengine.com/Datasheets/1/BNO055.pdf" H 8340 4040 50  0001 L CNN
@@
 Text GLabel 10200 1760 0    60   Input ~ 0
 Buzzer_ON_PD0
-Text GLabel 7726 2434 0    60   Output ~ 0
+Text GLabel 7786 2369 0    60   Output ~ 0
 5V_OUT
 Text GLabel 8725 1069 2    60   Output ~ 0
@@
 	7770 2283 7770 2284
 Wire Wire Line
-	7983 2153 7726 2434
+	7983 2153 7786 2369
 Wire Wire Line
 	8172 696  8167 651
@@
 $EndComp
 Wire Wire Line
-	4511 786  4681 786
+	4511 786  4516 786
 Wire Wire Line
 	4511 786  4341 781
@@
 	4341 1021 4331 1031
 Wire Wire Line
-	4116 1021 4281 1021
+	4116 1021 4121 1021
 Wire Wire Line
 	4116 1021 3827 1031
@@
 	10199 3777 10296 3777
 Wire Wire Line
-	1372 5212 1707 5212
-Wire Wire Line
-	2069 5214 2391 5214
+	1372 5212 1525 5212
+Wire Wire Line
+	2069 5214 2201 5214
 Wire Wire Line
 	2102 1652 2102 1867
@@
 L Cansat-rescue:Resistor 10K?
 U 1 1 5C719EFE
-P 8806 3372
-F 0 "10K?" V 8766 3552 60  0000 C CNN
-F 1 "Resistor" V 8641 3572 60  0000 C CNN
-F 2 "" H 8806 3372 60  0001 C CNN
-F 3 "" H 8806 3372 60  0001 C CNN
-	1    8806 3372
+P 8469 3353
+F 0 "10K?" H 8465 3485 60  0000 C CNN
+F 1 "Resistor" H 8483 3275 60  0000 C CNN
+F 2 "" H 8469 3353 60  0001 C CNN
+F 3 "" H 8469 3353 60  0001 C CNN
+	1    8469 3353
 	0    -1   -1   0
 $EndComp
@@
 L Cansat-rescue:Resistor 10K?
 U 1 1 5C719FFC
-P 8598 2612
-F 0 "10K?" V 8558 2792 60  0000 C CNN
-F 1 "Resistor" V 8433 2812 60  0000 C CNN
-F 2 "" H 8598 2612 60  0001 C CNN
-F 3 "" H 8598 2612 60  0001 C CNN
-	1    8598 2612
-	0    -1   -1   0
+P 8364 2942
+F 0 "10K?" H 8376 3040 60  0000 C CNN
+F 1 "Resistor" H 8376 2878 60  0000 C CNN
+F 2 "" H 8364 2942 60  0001 C CNN
+F 3 "" H 8364 2942 60  0001 C CNN
+	1    8364 2942
+	1    0    0    -1
 $EndComp
 $Comp
@@
 $EndComp
 $Comp
-L Cansat-rescue:Resistor 10K?
+L Cansat-rescue:Resistor 10K?opt
 U 1 1 5C71A18D
-P 6614 4396
-F 0 "10K?" V 6574 4576 60  0000 C CNN
-F 1 "Resistor" V 6449 4596 60  0000 C CNN
-F 2 "" H 6614 4396 60  0001 C CNN
-F 3 "" H 6614 4396 60  0001 C CNN
-	1    6614 4396
-	0    -1   -1   0
+P 7873 4807
+F 0 "10K?opt" H 7910 4709 60  0000 C CNN
+F 1 "Resistor" H 7952 4622 60  0000 C CNN
+F 2 "" H 7873 4807 60  0001 C CNN
+F 3 "" H 7873 4807 60  0001 C CNN
+	1    7873 4807
+	1    0    0    -1
 $EndComp
 Wire Wire Line
@@
 Wire Wire Line
 	6684 3740 6590 3740
+Text GLabel 6651 4071 0    50   Input ~ 0
+nBootLoadPin
+Wire Wire Line
+	6791 3840 6790 3840
+Wire Wire Line
+	6733 3840 6733 3901
+Wire Wire Line
+	6733 3901 6667 3901
+Wire Wire Line
+	6667 3901 6667 4071
+Wire Wire Line
+	6667 4071 6651 4071
+Connection ~ 6790 3840
+Wire Wire Line
+	6790 3840 6733 3840
+Wire Wire Line
+	8469 3433 8469 3637
+Wire Wire Line
+	8284 2942 8089 2942
+Wire Wire Line
+	8089 2942 8089 2944
+Wire Wire Line
+	8089 2944 8091 2944
+Wire Wire Line
+	8445 2943 8469 2942
+Wire Wire Line
+	8469 2942 8469 3273
+$Comp
+L power:+3.3V #PWR?
+U 1 1 5C723A8F
+P 8470 3092
+F 0 "#PWR?" H 8470 2942 50  0001 C CNN
+F 1 "+3.3V" V 8485 3220 50  0000 L CNN
+F 2 "" H 8470 3092 50  0001 C CNN
+F 3 "" H 8470 3092 50  0001 C CNN
+	1    8470 3092
+	0    1    1    0
+$EndComp
+Text GLabel 7698 4836 3    50   Input ~ 0
+nResetPin
+$Comp
+L power:+3.3V #PWR?
+U 1 1 5C72899A
+P 8148 4806
+F 0 "#PWR?" H 8148 4656 50  0001 C CNN
+F 1 "+3.3V" V 8163 4934 50  0000 L CNN
+F 2 "" H 8148 4806 50  0001 C CNN
+F 3 "" H 8148 4806 50  0001 C CNN
+	1    8148 4806
+	0    1    1    0
+$EndComp
+Wire Wire Line
+	7690 4640 7690 4837
+Wire Wire Line
+	7793 4837 7793 4808
+Wire Wire Line
+	7792 4807 7793 4807
+Wire Wire Line
+	8149 4807 8149 4806
+Connection ~ 8149 4807
+Wire Wire Line
+	8149 4807 8150 4807
+Wire Wire Line
+	7690 4837 7793 4837
+Wire Wire Line
+	7954 4807 8149 4807
+Wire Wire Line
+	7821 2330 7821 2331
+Connection ~ 4516 786
+Wire Wire Line
+	4516 786  4681 786
+Connection ~ 4121 1021
+Wire Wire Line
+	4121 1021 4281 1021
+Connection ~ 4282 1266
+Connection ~ 8451 2156
+Connection ~ 7983 2013
+Connection ~ 4118 1263
+Connection ~ 2104 1420
+Connection ~ 2103 1866
+Connection ~ 1372 5212
+Connection ~ 1525 5212
+Wire Wire Line
+	1525 5212 1707 5212
+Connection ~ 1883 5214
+Connection ~ 2071 5215
+Connection ~ 2201 5214
+Wire Wire Line
+	2201 5214 2391 5214
+Connection ~ 2390 5215
+Connection ~ 2636 4587
+Connection ~ 1853 2910
+Connection ~ 2370 2909
 $EndSCHEMATC

Commit message: and more touch up
Connections:
- wire segments 152 -> 151
Changed lines of the file:
@@
 	10666 6465 10666 6467
 Wire Wire Line
-	10199 3777 10296 3777
-Wire Wire Line
-	1372 5212 1525 5212
-Wire Wire Line
-	2069 5214 2201 5214
+	10199 3777 10253 3777
 Wire Wire Line
 	2102 1652 2102 1867
@@
 Wire Wire Line
 	7983 2153 7983 2151
-Text GLabel 9911 3776 3    50   Input ~ 0
+Text GLabel 9911 3775 3    50   Input ~ 0
 USART_RX_PC2
-Text GLabel 9996 3775 3    50   Output ~ 0
+Text GLabel 9995 3775 3    50   Output ~ 0
 USART_TX_PC3
 Text GLabel 3662 4441 0    60   Input ~ 0
@@
 Wire Wire Line
 	4121 1021 4281 1021
-Connection ~ 4282 1266
-Connection ~ 8451 2156
-Connection ~ 7983 2013
-Connection ~ 4118 1263
-Connection ~ 2104 1420
-Connection ~ 2103 1866
-Connection ~ 1372 5212
-Connection ~ 1525 5212
-Wire Wire Line
-	1525 5212 1707 5212
-Connection ~ 1883 5214
-Connection ~ 2071 5215
-Connection ~ 2201 5214
-Wire Wire Line
-	2201 5214 2391 5214
-Connection ~ 2390 5215
-Connection ~ 2636 4587
-Connection ~ 1853 2910
-Connection ~ 2370 2909
+Wire Wire Line
+	1372 5212 1707 5212
+Wire Wire Line
+	2069 5214 2391 5214
+Connection ~ 10253 3777
+Wire Wire Line
+	10253 3777 10296 3777
 $EndSCHEMATC

Commit message: Redid some symbols because of bug
added pdi and power supply circuit.
Parts:
- removed Fan_1_CTRL: 2N7002, Package_TO_SOT_SMD:SOT-23, symbol Transistor_FET:2N7002
- removed IC?: XBP9B-XCWT-001, XBP9BXCWT001, symbol Cansat-rescue:XBP9B-XCWT-001
- removed SNAP?: SERVO, symbol Cansat-rescue:SERVO
- removed SNAP?: FAN_0, symbol Cansat-rescue:FAN_0
- removed SNAP?: FAN_1, symbol Cansat-rescue:FAN_1
- removed comp?: VoltageDivider, voltage_divider, symbol Cansat-rescue:VoltageDivider
- added 100nF? (x3): C_Small, symbol Device:C_Small
- added C? (x3): uF0.1, symbol Device:C
- added C?: 0.1uF, symbol Device:C
- added C?: 10uF, symbol Device:CP1
- added IC?: XBP9B-XCWT-001, XBP9BXCWT001, symbol Cansat-rescue:XBP9B-XCWT-001
- added J? (x2): DC_Moter, symbol Connector_Generic:Conn_01x02
- added J?: PDI, symbol Connector_Generic:Conn_02x03_Top_Bottom
- added L?: INDUCTOR, symbol pspice:INDUCTOR
- added R?: R, symbol Device:R
- added R?: 10kohm, symbol Device:R
- added S?: Servo, symbol Cansat-rescue:Servo
Connections:
- net labels added: MCUAVCC, MCUGND, MCUGND2, MCUVCC, TCE0
- net labels removed: +5V, LED_ON_PE0, MOSFET_2
- wire segments 151 -> 185
- no-connect marks 0 -> 2
Other:
- moved on the sheet: 100nF, 10K, 10K?, 10K?opt, 10k, 4.7uF, 5VReg?, Bar-Pres-Sensor?, Breakout?, CoSel_SUS1R5, Fan_0_CTRL, GPS?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

Commit message: removed unecisisary capacitors
Parts:
- removed 100nF?: C_Small, symbol Device:C_Small
- removed C? (x3): uF0.1, symbol Device:C
- removed C?: 0.1uF, symbol Device:C
Connections:
- wire segments 185 -> 174
Changed lines of the file:
@@
 Text GLabel 4550 4500 3    50   Input ~ 0
 USART_RX_PD2
-Text GLabel 5150 3100 2    50   Output ~ 0
+Text GLabel 4950 3100 2    50   Output ~ 0
 USART_TX_PD3
-Text GLabel 1600 6550 0    50   Input ~ 0
+Text GLabel 2100 6350 0    50   Input ~ 0
 USART_RX_PD2
-Text GLabel 1600 6450 0    50   Output ~ 0
+Text GLabel 2100 6450 0    50   Output ~ 0
 USART_TX_PD3
 Text GLabel 4350 4500 3    50   Output ~ 0
@@
 $EndComp
 $Comp
-L Device:C C?
-U 1 1 5C88E6E0
-P 1800 6700
-F 0 "C?" H 1915 6746 50  0000 L CNN
-F 1 "uF0.1" H 1915 6655 50  0000 L CNN
-F 2 "" H 1838 6550 50  0001 C CNN
-F 3 "~" H 1800 6700 50  0001 C CNN
-	1    1800 6700
-	-1   0    0    1
-$EndComp
-$Comp
-L power:GND #PWR?
-U 1 1 5C88E78A
-P 1800 6850
-F 0 "#PWR?" H 1800 6600 50  0001 C CNN
-F 1 "GND" H 1805 6677 50  0000 C CNN
-F 2 "" H 1800 6850 50  0001 C CNN
-F 3 "" H 1800 6850 50  0001 C CNN
-	1    1800 6850
-	1    0    0    -1
-$EndComp
-$Comp
 L Device:R R?
 U 1 1 5C893CEA
@@
 Wire Wire Line
 	10650 6100 10800 6100
-Wire Wire Line
-	4950 3100 5050 3100
-$Comp
-L Device:C C?
-U 1 1 5C920859
-P 5050 2950
-F 0 "C?" H 4900 3050 50  0000 L CNN
-F 1 "0.1uF" H 5200 2950 50  0000 L CNN
-F 2 "" H 5088 2800 50  0001 C CNN
-F 3 "~" H 5050 2950 50  0001 C CNN
-	1    5050 2950
-	1    0    0    -1
-$EndComp
-Connection ~ 5050 3100
-Wire Wire Line
-	5050 3100 5150 3100
-$Comp
-L power:GND #PWR?
-U 1 1 5C920AC7
-P 5050 2800
-F 0 "#PWR?" H 5050 2550 50  0001 C CNN
-F 1 "GND" H 5050 2650 50  0000 C CNN
-F 2 "" H 5050 2800 50  0000 C CNN
-F 3 "" H 5050 2800 50  0000 C CNN
-	1    5050 2800
-	-1   0    0    1
-$EndComp
 $Comp
 L Cansat-rescue:XBP9B-XCWT-001 IC?
@@
 $EndComp
 $Comp
-L Device:C C?
-U 1 1 5C92CB12
-P 2050 6100
-F 0 "C?" H 1800 6200 50  0000 L CNN
-F 1 "uF0.1" H 1750 6100 50  0000 L CNN
-F 2 "" H 2088 5950 50  0001 C CNN
-F 3 "~" H 2050 6100 50  0001 C CNN
-	1    2050 6100
-	1    0    0    -1
-$EndComp
-$Comp
-L power:GND #PWR?
-U 1 1 5C92CCCE
-P 2050 5950
-F 0 "#PWR?" H 2050 5700 50  0001 C CNN
-F 1 "GND" H 2055 5777 50  0000 C CNN
-F 2 "" H 2050 5950 50  0001 C CNN
-F 3 "" H 2050 5950 50  0001 C CNN
-	1    2050 5950
-	-1   0    0    1
-$EndComp
-Wire Wire Line
-	1600 6550 1800 6550
-Wire Wire Line
-	1950 6550 1950 6350
-Wire Wire Line
-	1950 6350 2100 6350
-Wire Wire Line
-	1950 6250 2050 6250
-Connection ~ 1800 6550
-Wire Wire Line
-	1800 6550 1950 6550
-Connection ~ 2050 6250
-Wire Wire Line
-	2050 6250 2100 6250
-Wire Wire Line
-	1600 6450 1650 6450
-$Comp
-L Device:C C?
-U 1 1 5C93B75B
-P 1650 6300
-F 0 "C?" H 1400 6400 50  0000 L CNN
-F 1 "uF0.1" H 1350 6300 50  0000 L CNN
-F 2 "" H 1688 6150 50  0001 C CNN
-F 3 "~" H 1650 6300 50  0001 C CNN
-	1    1650 6300
-	1    0    0    -1
-$EndComp
-Connection ~ 1650 6450
-Wire Wire Line
-	1650 6450 2100 6450
-$Comp
-L power:GND #PWR?
-U 1 1 5C93B7D1
-P 1650 6150
-F 0 "#PWR?" H 1650 5900 50  0001 C CNN
-F 1 "GND" H 1655 5977 50  0000 C CNN
-F 2 "" H 1650 6150 50  0001 C CNN
-F 3 "" H 1650 6150 50  0001 C CNN
-	1    1650 6150
-	-1   0    0    1
-$EndComp
-$Comp
 L Device:CP1 C?
 U 1 1 5C943F8C
@@
 	-1   0    0    1
 $EndComp
-Text GLabel 10100 6150 3    50   Input ~ 0
+Text GLabel 10100 5600 3    50   Input ~ 0
 TCE0
-Wire Wire Line
-	10100 5600 10100 6000
-$Comp
-L Device:C_Small 100nF?
-U 1 1 5CA380E7
-P 10000 6000
-F 0 "100nF?" V 9771 6000 50  0000 C CNN
-F 1 "C_Small" V 9862 6000 50  0000 C CNN
-F 2 "" H 10000 6000 50  0001 C CNN
-F 3 "~" H 10000 6000 50  0001 C CNN
-	1    10000 6000
-	0    -1   -1   0
-$EndComp
-Connection ~ 10100 6000
-Wire Wire Line
-	10100 6000 10100 6150
-$Comp
-L power:GND #PWR?
-U 1 1 5CA381BE
-P 9900 6000
-F 0 "#PWR?" H 9900 5750 50  0001 C CNN
-F 1 "GND" H 9905 5827 50  0000 C CNN
-F 2 "" H 9900 6000 50  0001 C CNN
-F 3 "" H 9900 6000 50  0001 C CNN
-	1    9900 6000
-	0    1    1    0
-$EndComp
 Text GLabel 4950 3600 2    50   Input ~ 0
 TCE0
+Wire Wire Line
+	1950 6250 2100 6250
 $EndSCHEMATC
